File: PI0E.brd (EAGLE design)
At the start: 36 parts, among them T1 WE-LAN-10/100/1000-BASE-T,749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, X1 22-23-2021, X2 22-23-2021

Commit message: cleaning traces
Routing:
- net 3: track 23.4 -> 21.1 mm
- net 6: track 19.1 -> 17.5 mm
Changed lines of the file:
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@@
 <wire x1="68.7356" y1="25.708" x2="68.7578" y2="25.7302" width="0.4064" layer="1"/>
 <via x="68.7578" y="25.7302" extent="1-16" drill="0.6"/>
-<wire x1="68.7578" y1="25.7302" x2="71.6661" y2="25.7302" width="0.4064" layer="16"/>
-<wire x1="71.6661" y1="25.7302" x2="71.7042" y2="25.6921" width="0.4064" layer="16"/>
-<via x="71.7042" y="25.6921" extent="1-16" drill="0.6"/>
-<wire x1="71.7042" y1="25.6921" x2="71.7042" y2="17.3609" width="0.4064" layer="1"/>
+<wire x1="68.7578" y1="25.7302" x2="70.8791" y2="23.6082" width="0.4064" layer="16"/>
+<wire x1="70.8791" y1="23.6082" x2="71.7042" y2="22.8271" width="0.4064" layer="16"/>
+<via x="71.7042" y="22.8271" extent="1-16" drill="0.6"/>
+<wire x1="71.7042" y1="22.8271" x2="71.7042" y2="17.3609" width="0.4064" layer="1"/>
 <wire x1="71.7042" y1="17.3609" x2="73.4441" y2="15.621" width="0.4064" layer="1"/>
 <wire x1="73.4441" y1="15.621" x2="74.3458" y2="15.621" width="0.4064" layer="1"/>
@@
 <contactref element="ENC28J60" pad="5"/>
 <wire x1="20.755" y1="6.445" x2="20.755" y2="4.274" width="0.254" layer="1"/>
-<wire x1="20.755" y1="4.274" x2="20.4975" y2="3.7774" width="0.254" layer="1"/>
-<via x="20.4975" y="3.7774" extent="1-16" drill="0.6096"/>
-<wire x1="20.4975" y1="3.7774" x2="20.816" y2="4.301" width="0.254" layer="16"/>
+<wire x1="20.755" y1="4.274" x2="20.4975" y2="3.7664" width="0.254" layer="1"/>
+<via x="20.4975" y="3.7664" extent="1-16" drill="0.6096"/>
+<wire x1="20.4975" y1="3.7664" x2="20.816" y2="4.301" width="0.254" layer="16"/>
 <wire x1="20.816" y1="4.301" x2="20.828" y2="8.636" width="0.254" layer="16"/>
 <wire x1="20.828" y1="8.636" x2="23.876" y2="11.684" width="0.254" layer="16"/>
@@
 <contactref element="ENC28J60" pad="24"/>
 <contactref element="ENC28J60" pad="21"/>
-<wire x1="17.443459375" y1="9.956540625" x2="17.255" y2="9.945" width="0.4064" layer="1"/>
+<wire x1="17.443459375" y1="9.956540625" x2="17.255" y2="9.945" width="0.254" layer="1"/>
 <contactref element="TLV1137" pad="4"/>
 <contactref element="C11" pad="1"/>
@@
 <wire x1="75.942" y1="15.3329" x2="74.8792" y2="16.3957" width="0.4064" layer="1"/>
 <wire x1="74.8792" y1="16.3957" x2="73.8378" y2="16.3957" width="0.4064" layer="1"/>
-<wire x1="73.8378" y1="16.3957" x2="73.39965" y2="16.83385" width="0.4064" layer="1"/>
-<wire x1="73.39965" y1="16.83385" x2="73.0504" y2="17.1831" width="0.4064" layer="1"/>
+<wire x1="73.8378" y1="16.3957" x2="72.9234" y2="17.3101" width="0.4064" layer="1"/>
 <wire x1="66.01" y1="28.741" x2="68.8331" y2="28.741" width="0.4064" layer="1"/>
 <wire x1="68.8331" y1="28.741" x2="68.8467" y2="28.7274" width="0.4064" layer="1"/>
 <via x="68.8467" y="28.7274" extent="1-16" drill="0.6"/>
-<wire x1="68.8467" y1="28.7274" x2="72.9234" y2="28.7274" width="0.4064" layer="16"/>
-<via x="72.9234" y="28.7274" extent="1-16" drill="0.6"/>
-<wire x1="72.9234" y1="28.7274" x2="72.9234" y2="17.3101" width="0.4064" layer="1"/>
-<wire x1="72.9234" y1="17.3101" x2="73.0504" y2="17.1831" width="0.4064" layer="1"/>
+<wire x1="68.8467" y1="28.7274" x2="72.9234" y2="24.7414" width="0.4064" layer="16"/>
+<via x="72.9234" y="24.7414" extent="1-16" drill="0.6"/>
+<wire x1="72.9234" y1="24.7414" x2="72.9234" y2="17.3101" width="0.4064" layer="1"/>
 </signal>
 <signal name="N$22">
@@
 <wire x1="21.348" y1="4.7107" x2="21.3474" y2="4.5161" width="0.254" layer="1"/>
 <wire x1="21.3474" y1="4.5161" x2="21.352" y2="3.616" width="0.254" layer="1"/>
-<wire x1="21.352" y1="3.616" x2="21.358" y2="3.23" width="0.254" layer="1"/>
-<wire x1="21.358" y1="3.23" x2="20.965" y2="2.882" width="0.254" layer="1"/>
-<wire x1="20.965" y1="2.882" x2="20.6509" y2="2.5596" width="0.254" layer="1"/>
-<via x="20.6509" y="2.5596" extent="1-16" drill="0.6096"/>
-<wire x1="20.6509" y1="2.5596" x2="21.284" y2="3.091" width="0.254" layer="16"/>
+<wire x1="21.352" y1="3.616" x2="21.358" y2="3.133" width="0.254" layer="1"/>
+<wire x1="21.358" y1="3.133" x2="20.976" y2="2.709" width="0.254" layer="1"/>
+<wire x1="20.976" y1="2.709" x2="20.882" y2="2.5982" width="0.254" layer="1"/>
+<via x="20.882" y="2.5982" extent="1-16" drill="0.6096"/>
+<wire x1="20.882" y1="2.5982" x2="21.284" y2="3.091" width="0.254" layer="16"/>
 <wire x1="21.284" y1="3.091" x2="21.346" y2="3.194" width="0.254" layer="16"/>
 <wire x1="21.346" y1="3.194" x2="21.339" y2="4.008" width="0.254" layer="16"/>
